Commit message: 7th commit

File: mintchoco1_description/urdf/mintchoco1.urdf.xacro (robot description, xacro)
@@ -2,10 +2,10 @@
 <robot name="mintchoco1" xmlns:xacro="http://ros.org/wiki/xacro">
   <!-- Fix the base_link -->
-  <!--link name="world"/-->
-  <!--joint name="fixed" type="fixed">
+  <link name="world"/>
+  <joint name="fixed" type="fixed">
     <parent link="world"/>
     <child link="base_link"/>
      <origin xyz="0.0 0.0 0.005" rpy="0 0 0" />
-  </joint-->
+  </joint>
   <link name="base_link">
     <inertial>
@@ -275,5 +275,5 @@
       link="RF_link1" />
     <axis
-      xyz="-0.99999 0 0.005102" />
+      xyz="0.99999 0 0.005102" />
     <limit
       lower="-3.14"
@@ -452,5 +452,5 @@
       link="LB_link1" />
     <axis
-      xyz="0.99995 0 -0.010204" />
+      xyz="-0.99995 0 -0.010204" />
     <limit
       lower="-3.14"
@@ -629,5 +629,5 @@
       link="RB_link1" />
     <axis
-      xyz="0.99999 0 -0.005102" />
+      xyz="0.99999 0 0.005102" />
     <limit
       lower="-3.14"
@@ -747,5 +747,5 @@
       link="RB_link3" />
     <axis
-      xyz="1 0.0017021 0" />
+      xyz="-1 0.0017021 0" />
     <limit
       lower="-3.14"
