Commit message: second commit

File: mintchoco1_description/urdf/mintchoco1.gazebo.xacro (robot description, xacro)
@@ -10,43 +10,121 @@
 <!-- Base_link : Black -->
   <gazebo reference="base_link">
+    <kp>1000000.0</kp>
+    <kd>1.0</kd>
+    <mu1>0.8</mu1>
+    <mu2>0.8</mu2>
+    <maxVel>0.0</maxVel>
+    <minDepth>0.001</minDepth>
     <material>Gazebo/DarkGrey</material>
   </gazebo>
 <!-- Link1 : Black -->
   <gazebo reference="LF_link1">
+    <kp>1000000.0</kp>
+    <kd>1.0</kd>
+    <mu1>0.8</mu1>
+    <mu2>0.8</mu2>
+    <maxVel>0.0</maxVel>
+    <minDepth>0.001</minDepth>
     <material>Gazebo/DarkGrey</material>
   </gazebo>
   <gazebo reference="LB_link1">
+    <kp>1000000.0</kp>
+    <kd>1.0</kd>
+    <mu1>0.8</mu1>
+    <mu2>0.8</mu2>
+    <maxVel>0.0</maxVel>
+    <minDepth>0.001</minDepth>
     <material>Gazebo/DarkGrey</material>
   </gazebo>
   <gazebo reference="RF_link1">
+    <kp>1000000.0</kp>
+    <kd>1.0</kd>
+    <mu1>0.8</mu1>
+    <mu2>0.8</mu2>
+    <maxVel>0.0</maxVel>
+    <minDepth>0.001</minDepth>
     <material>Gazebo/DarkGrey</material>
   </gazebo>
   <gazebo reference="RB_link1">
+    <kp>1000000.0</kp>
+    <kd>1.0</kd>
+    <mu1>0.8</mu1>
+    <mu2>0.8</mu2>
+    <maxVel>0.0</maxVel>
+    <minDepth>0.001</minDepth>
     <material>Gazebo/DarkGrey</material>
   </gazebo>
 <!-- Link2 : Red -->
   <gazebo reference="LF_link2">
+    <kp>1000000.0</kp>
+    <kd>1.0</kd>
+    <mu1>0.8</mu1>
+    <mu2>0.8</mu2>
+    <maxVel>0.0</maxVel>
+    <minDepth>0.001</minDepth>
     <material>Gazebo/RedBright</material>
   </gazebo>
   <gazebo reference="LB_link2">
+    <kp>1000000.0</kp>
+    <kd>1.0</kd>
+    <mu1>0.8</mu1>
+    <mu2>0.8</mu2>
+    <maxVel>0.0</maxVel>
+    <minDepth>0.001</minDepth>
     <material>Gazebo/RedBright</material>
   </gazebo>
   <gazebo reference="RF_link2">
+    <kp>1000000.0</kp>
+    <kd>1.0</kd>
+    <mu1>0.8</mu1>
+    <mu2>0.8</mu2>
+    <maxVel>0.0</maxVel>
+    <minDepth>0.001</minDepth>
     <material>Gazebo/RedBright</material>
   </gazebo>
   <gazebo reference="RB_link2">
+    <kp>1000000.0</kp>
+    <kd>1.0</kd>
+    <mu1>0.8</mu1>
+    <mu2>0.8</mu2>
+    <maxVel>0.0</maxVel>
+    <minDepth>0.001</minDepth>
     <material>Gazebo/RedBright</material>
   </gazebo>
 <!-- Link3 : DarkGrey -->
   <gazebo reference="LF_link3">
+    <kp>1000000.0</kp>
+    <kd>1.0</kd>
+    <mu1>0.8</mu1>
+    <mu2>0.8</mu2>
+    <maxVel>0.0</maxVel>
+    <minDepth>0.001</minDepth>
     <material>Gazebo/DarkGrey</material>
   </gazebo>
   <gazebo reference="LB_link3">
+    <kp>1000000.0</kp>
+    <kd>1.0</kd>
+    <mu1>0.8</mu1>
+    <mu2>0.8</mu2>
+    <maxVel>0.0</maxVel>
+    <minDepth>0.001</minDepth>
     <material>Gazebo/DarkGrey</material>
   </gazebo>
   <gazebo reference="RF_link3">
+    <kp>1000000.0</kp>
+    <kd>1.0</kd>
+    <mu1>0.8</mu1>
+    <mu2>0.8</mu2>
+    <maxVel>0.0</maxVel>
+    <minDepth>0.001</minDepth>
     <material>Gazebo/DarkGrey</material>
   </gazebo>
   <gazebo reference="RB_link3">
+    <kp>1000000.0</kp>
+    <kd>1.0</kd>
+    <mu1>0.8</mu1>
+    <mu2>0.8</mu2>
+    <maxVel>0.0</maxVel>
+    <minDepth>0.001</minDepth>
     <material>Gazebo/DarkGrey</material>
   </gazebo>

File: mintchoco1_description/urdf/mintchoco1.transmission.xacro (robot description, xacro)
@@ -1,4 +1,4 @@
 <?xml version="1.0"?>
-<robot name="mintch0co1" xmlns:xacro="http://ros.org/wiki/xacro">
+<robot name="mintchoco1" xmlns:xacro="http://ros.org/wiki/xacro">
 <!-- joint1 Transmission -->
   <transmission name="LF_joint1">

File: mintchoco1_description/urdf/mintchoco1.urdf.xacro (robot description, xacro)
@@ -2,10 +2,10 @@
 <robot name="mintchoco1" xmlns:xacro="http://ros.org/wiki/xacro">
   <!-- Fix the base_link -->
-  <link name="world"/>
-  <joint name="fixed" type="fixed">
+  <!--link name="world"/-->
+  <!--joint name="fixed" type="fixed">
     <parent link="world"/>
     <child link="base_link"/>
      <origin xyz="0.0 0.0 0.005" rpy="0 0 0" />
-  </joint>
+  </joint-->
   <link name="base_link">
     <inertial>
@@ -102,6 +102,7 @@
       lower="-3.14"
       upper="3.14"
-      effort="0"
-      velocity="0" />
+      effort="1"
+      velocity="4.8" />
+    <!--dynamics damping ="0.7"/-->
   </joint>
   <link
@@ -160,6 +161,7 @@
       lower="-3.14"
       upper="3.14"
-      effort="0"
-      velocity="0" />
+      effort="1"
+      velocity="4.8" />
+    <!--dynamics damping ="0.7"/-->
   </joint>
   <link
@@ -218,6 +220,7 @@
       lower="-3.14"
       upper="3.14"
-      effort="0"
-      velocity="0" />
+      effort="1"
+      velocity="4.8" />
+    <!--dynamics damping ="0.7"/-->
   </joint>
   <link
@@ -276,6 +279,7 @@
       lower="-3.14"
       upper="3.14"
-      effort="0"
-      velocity="0" />
+      effort="1"
+      velocity="4.8" />
+    <!--dynamics damping ="0.7"/-->
   </joint>
   <link
@@ -334,6 +338,7 @@
       lower="-3.14"
       upper="3.14"
-      effort="0"
-      velocity="0" />
+      effort="1"
+      velocity="4.8" />
+    <!--dynamics damping ="0.7"/-->
   </joint>
   <link
@@ -392,6 +397,7 @@
       lower="-3.14"
       upper="3.14"
-      effort="0"
-      velocity="0" />
+      effort="1"
+      velocity="4.8" />
+    <!--dynamics damping ="0.7"/-->
   </joint>
   <link
@@ -450,6 +456,7 @@
       lower="-3.14"
       upper="3.14"
-      effort="0"
-      velocity="0" />
+      effort="1"
+      velocity="4.8" />
+    <!--dynamics damping ="0.7"/-->
   </joint>
   <link
@@ -508,6 +515,7 @@
       lower="-3.14"
       upper="3.14"
-      effort="0"
-      velocity="0" />
+      effort="1"
+      velocity="4.8" />
+    <!--dynamics damping ="0.7"/-->
   </joint>
   <link
@@ -566,6 +574,7 @@
       lower="-3.14"
       upper="3.14"
-      effort="0"
-      velocity="0" />
+      effort="1"
+      velocity="4.8" />
+    <!--dynamics damping ="0.7"/-->
   </joint>
   <link
@@ -624,6 +633,7 @@
       lower="-3.14"
       upper="3.14"
-      effort="0"
-      velocity="0" />
+      effort="1"
+      velocity="4.8" />
+    <!--dynamics damping ="0.7"/-->
   </joint>
   <link
@@ -682,6 +692,7 @@
       lower="-3.14"
       upper="3.14"
-      effort="0"
-      velocity="0" />
+      effort="1"
+      velocity="4.8" />
+    <!--dynamics damping ="0.7"/-->
   </joint>
   <link
@@ -740,6 +751,7 @@
       lower="-3.14"
       upper="3.14"
-      effort="0"
-      velocity="0" />
+      effort="1"
+      velocity="4.8" />
+    <!--dynamics damping ="0.7"/-->
   </joint>
 </robot>

Commit message: 10th commit

File: mintchoco1_description/urdf/mintchoco1.gazebo.xacro (robot description, xacro)
@@ -11,9 +11,10 @@
   <gazebo reference="base_link">
     <kp>1000000.0</kp>
-    <kd>1.0</kd>
-    <mu1>0.8</mu1>
-    <mu2>0.8</mu2>
-    <maxVel>0.0</maxVel>
+    <kd>50.0</kd>
+    <mu1>0.1</mu1>
+    <mu2>0.1</mu2>
+    <maxVel>1.0</maxVel>
     <minDepth>0.001</minDepth>
+    <fdir1>0 0 0</fdir1>
     <material>Gazebo/DarkGrey</material>
   </gazebo>
@@ -21,36 +22,40 @@
   <gazebo reference="LF_link1">
     <kp>1000000.0</kp>
-    <kd>1.0</kd>
-    <mu1>0.8</mu1>
-    <mu2>0.8</mu2>
-    <maxVel>0.0</maxVel>
+    <kd>50.0</kd>
+    <mu1>0.1</mu1>
+    <mu2>0.1</mu2>
+    <maxVel>1.0</maxVel>
     <minDepth>0.001</minDepth>
+    <fdir1>0 0 0</fdir1>
     <material>Gazebo/DarkGrey</material>
   </gazebo>
   <gazebo reference="LB_link1">
     <kp>1000000.0</kp>
-    <kd>1.0</kd>
-    <mu1>0.8</mu1>
-    <mu2>0.8</mu2>
-    <maxVel>0.0</maxVel>
+    <kd>50.0</kd>
+    <mu1>0.1</mu1>
+    <mu2>0.1</mu2>
+    <maxVel>1.0</maxVel>
     <minDepth>0.001</minDepth>
+    <fdir1>0 0 0</fdir1>
     <material>Gazebo/DarkGrey</material>
   </gazebo>
   <gazebo reference="RF_link1">
     <kp>1000000.0</kp>
-    <kd>1.0</kd>
-    <mu1>0.8</mu1>
-    <mu2>0.8</mu2>
-    <maxVel>0.0</maxVel>
+    <kd>50.0</kd>
+    <mu1>0.1</mu1>
+    <mu2>0.1</mu2>
+    <maxVel>1.0</maxVel>
     <minDepth>0.001</minDepth>
+    <fdir1>0 0 0</fdir1>
     <material>Gazebo/DarkGrey</material>
   </gazebo>
   <gazebo reference="RB_link1">
     <kp>1000000.0</kp>
-    <kd>1.0</kd>
-    <mu1>0.8</mu1>
-    <mu2>0.8</mu2>
-    <maxVel>0.0</maxVel>
+    <kd>50.0</kd>
+    <mu1>0.1</mu1>
+    <mu2>0.1</mu2>
+    <maxVel>1.0</maxVel>
     <minDepth>0.001</minDepth>
+    <fdir1>0 0 0</fdir1>
     <material>Gazebo/DarkGrey</material>
   </gazebo>
@@ -58,36 +63,40 @@
   <gazebo reference="LF_link2">
     <kp>1000000.0</kp>
-    <kd>1.0</kd>
-    <mu1>0.8</mu1>
-    <mu2>0.8</mu2>
-    <maxVel>0.0</maxVel>
+    <kd>50.0</kd>
+    <mu1>0.1</mu1>
+    <mu2>0.1</mu2>
+    <maxVel>1.0</maxVel>
     <minDepth>0.001</minDepth>
+    <fdir1>0 0 0</fdir1>
     <material>Gazebo/RedBright</material>
   </gazebo>
   <gazebo reference="LB_link2">
     <kp>1000000.0</kp>
-    <kd>1.0</kd>
-    <mu1>0.8</mu1>
-    <mu2>0.8</mu2>
-    <maxVel>0.0</maxVel>
+    <kd>50.0</kd>
+    <mu1>0.1</mu1>
+    <mu2>0.1</mu2>
+    <maxVel>1.0</maxVel>
     <minDepth>0.001</minDepth>
+    <fdir1>0 0 0</fdir1>
     <material>Gazebo/RedBright</material>
   </gazebo>
   <gazebo reference="RF_link2">
     <kp>1000000.0</kp>
-    <kd>1.0</kd>
-    <mu1>0.8</mu1>
-    <mu2>0.8</mu2>
-    <maxVel>0.0</maxVel>
+    <kd>50.0</kd>
+    <mu1>0.1</mu1>
+    <mu2>0.1</mu2>
+    <maxVel>1.1</maxVel>
     <minDepth>0.001</minDepth>
+    <fdir1>0 0 0</fdir1>
     <material>Gazebo/RedBright</material>
   </gazebo>
   <gazebo reference="RB_link2">
     <kp>1000000.0</kp>
-    <kd>1.0</kd>
-    <mu1>0.8</mu1>
-    <mu2>0.8</mu2>
-    <maxVel>0.0</maxVel>
+    <kd>50.0</kd>
+    <mu1>0.1</mu1>
+    <mu2>0.1</mu2>
+    <maxVel>1.0</maxVel>
     <minDepth>0.001</minDepth>
+    <fdir1>0 0 0</fdir1>
     <material>Gazebo/RedBright</material>
   </gazebo>
@@ -95,36 +104,40 @@
   <gazebo reference="LF_link3">
     <kp>1000000.0</kp>
-    <kd>1.0</kd>
-    <mu1>0.8</mu1>
-    <mu2>0.8</mu2>
-    <maxVel>0.0</maxVel>
+    <kd>50.0</kd>
+    <mu1>0.1</mu1>
+    <mu2>0.1</mu2>
+    <maxVel>1.0</maxVel>
     <minDepth>0.001</minDepth>
+    <fdir1>0 0 0</fdir1>
     <material>Gazebo/DarkGrey</material>
   </gazebo>
   <gazebo reference="LB_link3">
     <kp>1000000.0</kp>
-    <kd>1.0</kd>
-    <mu1>0.8</mu1>
-    <mu2>0.8</mu2>
-    <maxVel>0.0</maxVel>
+    <kd>50.0</kd>
+    <mu1>0.1</mu1>
+    <mu2>0.1</mu2>
+    <maxVel>1.0</maxVel>
     <minDepth>0.001</minDepth>
+    <fdir1>0 0 0</fdir1>
     <material>Gazebo/DarkGrey</material>
   </gazebo>
   <gazebo reference="RF_link3">
     <kp>1000000.0</kp>
-    <kd>1.0</kd>
-    <mu1>0.8</mu1>
-    <mu2>0.8</mu2>
-    <maxVel>0.0</maxVel>
+    <kd>50.0</kd>
+    <mu1>0.1</mu1>
+    <mu2>0.1</mu2>
+    <maxVel>1.0</maxVel>
     <minDepth>0.001</minDepth>
+    <fdir1>0 0 0</fdir1>
     <material>Gazebo/DarkGrey</material>
   </gazebo>
   <gazebo reference="RB_link3">
     <kp>1000000.0</kp>
-    <kd>1.0</kd>
-    <mu1>0.8</mu1>
-    <mu2>0.8</mu2>
-    <maxVel>0.0</maxVel>
+    <kd>50.0</kd>
+    <mu1>0.1</mu1>
+    <mu2>0.1</mu2>
+    <maxVel>1.0</maxVel>
     <minDepth>0.001</minDepth>
+    <fdir1>0 0 0</fdir1>
     <material>Gazebo/DarkGrey</material>
   </gazebo>

File: mintchoco1_description/urdf/mintchoco1.urdf.xacro (robot description, xacro)
@@ -3,8 +3,8 @@
   <!-- Fix the base_link -->
   <link name="world"/>
-  <joint name="fixed" type="fixed">
+  <joint name="planar" type="planar">
     <parent link="world"/>
     <child link="base_link"/>
-     <origin xyz="0.0 0.0 0.005" rpy="0 0 0" />
+     <origin xyz="0.0 0.0 0.0" rpy="0 0 0" />
   </joint>
   <link name="base_link">
@@ -102,5 +102,5 @@
       lower="-3.14"
       upper="3.14"
-      effort="1"
+      effort="10"
       velocity="4.8" />
     <!--dynamics damping ="0.7"/-->
@@ -161,5 +161,5 @@
       lower="-3.14"
       upper="3.14"
-      effort="1"
+      effort="10"
       velocity="4.8" />
     <!--dynamics damping ="0.7"/-->
@@ -220,5 +220,5 @@
       lower="-3.14"
       upper="3.14"
-      effort="1"
+      effort="10"
       velocity="4.8" />
     <!--dynamics damping ="0.7"/-->
@@ -279,5 +279,5 @@
       lower="-3.14"
       upper="3.14"
-      effort="1"
+      effort="10"
       velocity="4.8" />
     <!--dynamics damping ="0.7"/-->
@@ -338,5 +338,5 @@
       lower="-3.14"
       upper="3.14"
-      effort="1"
+      effort="10"
       velocity="4.8" />
     <!--dynamics damping ="0.7"/-->
@@ -397,5 +397,5 @@
       lower="-3.14"
       upper="3.14"
-      effort="1"
+      effort="10"
       velocity="4.8" />
     <!--dynamics damping ="0.7"/-->
@@ -456,5 +456,5 @@
       lower="-3.14"
       upper="3.14"
-      effort="1"
+      effort="10"
       velocity="4.8" />
     <!--dynamics damping ="0.7"/-->
@@ -515,5 +515,5 @@
       lower="-3.14"
       upper="3.14"
-      effort="1"
+      effort="10"
       velocity="4.8" />
     <!--dynamics damping ="0.7"/-->
@@ -574,5 +574,5 @@
       lower="-3.14"
       upper="3.14"
-      effort="1"
+      effort="10"
       velocity="4.8" />
     <!--dynamics damping ="0.7"/-->
@@ -633,5 +633,5 @@
       lower="-3.14"
       upper="3.14"
-      effort="1"
+      effort="10"
       velocity="4.8" />
     <!--dynamics damping ="0.7"/-->
@@ -692,5 +692,5 @@
       lower="-3.14"
       upper="3.14"
-      effort="1"
+      effort="10"
       velocity="4.8" />
     <!--dynamics damping ="0.7"/-->
@@ -751,5 +751,5 @@
       lower="-3.14"
       upper="3.14"
-      effort="1"
+      effort="10"
       velocity="4.8" />
     <!--dynamics damping ="0.7"/-->

File: mintchoco1_description/urdf/mintchoco1_robot.urdf.xacro (robot description, xacro)
@@ -8,4 +8,4 @@
   <xacro:include filename="$(find mintchoco1_description)/urdf/mintchoco1.transmission.xacro" />
   <!-- Import URDF -->
-  <xacro:include filename="$(find mintchoco1_description)/urdf/mintchoco1.urdf.xacro" />
+  <xacro:include filename="$(find mintchoco1_description)/urdf/mintchoco1.urdf2.xacro" />
 </robot>

Commit message: commit 11

File: mintchoco1_description/urdf/mintchoco1.gazebo.xacro (robot description, xacro)
@@ -7,4 +7,25 @@
       <robotSimType>gazebo_ros_control/DefaultRobotHWSim</robotSimType>
     </plugin>
+  </gazebo>
+  <!-- imu plugin -->
+  <gazebo reference="imu_link">
+    <gravity>true</gravity>
+    <sensor name="imu_sensor" type="imu">
+      <always_on>true</always_on>
+      <update_rate>100</update_rate>
+      <visualize>true</visualize>
+      <topic>__default_topic__</topic>
+      <plugin filename="libgazebo_ros_imu_sensor.so" name="imu_plugin">
+        <topicName>imu</topicName>
+        <bodyName>imu_link</bodyName>
+        <updateRateHZ>10.0</updateRateHZ>
+        <gaussianNoise>0.0</gaussianNoise>
+        <xyzOffset>0 0 0</xyzOffset>
+        <rpyOffset>0 0 0</rpyOffset>
+        <frameName>imu_link</frameName>
+        <initialOrientationAsReference>false</initialOrientationAsReference>
+      </plugin>
+      <pose>0 0 0 0 0 0</pose>
+    </sensor>
   </gazebo>
 <!-- Base_link : Black -->
@@ -142,3 +163,27 @@
     <material>Gazebo/DarkGrey</material>
   </gazebo>
+  <xacro:macro name="RefJoint" params="ref">
+    <gazebo reference="${ref}">
+      <provideFeedback>true</provideFeedback>
+    </gazebo>
+  </xacro:macro>
+  <xacro:macro name="RefJoint" params="ref">
+    <plugin name="ft_sensor" filename="libgazebo_ros_ft_sensor.so">
+        <updateRate>100.0</updateRate>
+        <topicName>ft_sensor_topic</topicName>
+        <jointName>${ref}</jointName>
+    </plugin>
+  </xacro:macro>
+  <RefJoint ref="LF_joint1"/>
+  <RefJoint ref="LF_joint2"/>
+  <RefJoint ref="LF_joint3"/>
+  <RefJoint ref="LB_joint1"/>
+  <RefJoint ref="LB_joint2"/>
+  <RefJoint ref="LB_joint3"/>
+  <RefJoint ref="RF_joint1"/>
+  <RefJoint ref="RF_joint2"/>
+  <RefJoint ref="RF_joint3"/>
+  <RefJoint ref="RB_joint1"/>
+  <RefJoint ref="RB_joint2"/>
+  <RefJoint ref="RB_joint3"/>
 </robot>

File: mintchoco1_description/urdf/mintchoco1.urdf2.xacro (robot description, xacro)
@@ -2,4 +2,10 @@
 <robot name="mintchoco1" xmlns:xacro="http://ros.org/wiki/xacro">
   <xacro:include filename="$(find mintchoco1_description)/urdf/properties.urdf.xacro" />
+  <joint name="imu_joint" type="fixed">
+    <parent link="base_link"/>
+    <child link="imu_link"/>
+    <origin xyz="0.0 0.0 0.0" rpy="0 0 0"/>
+  </joint>
+  <link name="imu_link"/>
   <!-- Fix the base_link -->
   <link name="world"/>

Commit message: commit 13

File: mintchoco1_description/urdf/mintchoco1.gazebo.xacro (robot description, xacro)
@@ -40,127 +40,40 @@
     <material>Gazebo/DarkGrey</material>
   </gazebo>
-<!-- Link1 : Black -->
-  <gazebo reference="LF_link1">
-    <kp>1000000.0</kp>
-    <kd>50.0</kd>
-    <mu1>0.1</mu1>
-    <mu2>0.1</mu2>
-    <maxVel>1.0</maxVel>
-    <minDepth>0.001</minDepth>
-    <fdir1>0 0 0</fdir1>
-    <material>Gazebo/DarkGrey</material>
-  </gazebo>
-  <gazebo reference="LB_link1">
-    <kp>1000000.0</kp>
-    <kd>50.0</kd>
-    <mu1>0.1</mu1>
-    <mu2>0.1</mu2>
-    <maxVel>1.0</maxVel>
-    <minDepth>0.001</minDepth>
-    <fdir1>0 0 0</fdir1>
-    <material>Gazebo/DarkGrey</material>
-  </gazebo>
-  <gazebo reference="RF_link1">
-    <kp>1000000.0</kp>
-    <kd>50.0</kd>
-    <mu1>0.1</mu1>
-    <mu2>0.1</mu2>
-    <maxVel>1.0</maxVel>
-    <minDepth>0.001</minDepth>
-    <fdir1>0 0 0</fdir1>
-    <material>Gazebo/DarkGrey</material>
-  </gazebo>
-  <gazebo reference="RB_link1">
-    <kp>1000000.0</kp>
-    <kd>50.0</kd>
-    <mu1>0.1</mu1>
-    <mu2>0.1</mu2>
-    <maxVel>1.0</maxVel>
-    <minDepth>0.001</minDepth>
-    <fdir1>0 0 0</fdir1>
-    <material>Gazebo/DarkGrey</material>
-  </gazebo>
-<!-- Link2 : Red -->
-  <gazebo reference="LF_link2">
-    <kp>1000000.0</kp>
-    <kd>50.0</kd>
-    <mu1>0.1</mu1>
-    <mu2>0.1</mu2>
-    <maxVel>1.0</maxVel>
-    <minDepth>0.001</minDepth>
-    <fdir1>0 0 0</fdir1>
-    <material>Gazebo/RedBright</material>
-  </gazebo>
-  <gazebo reference="LB_link2">
-    <kp>1000000.0</kp>
-    <kd>50.0</kd>
-    <mu1>0.1</mu1>
-    <mu2>0.1</mu2>
-    <maxVel>1.0</maxVel>
-    <minDepth>0.001</minDepth>
-    <fdir1>0 0 0</fdir1>
-    <material>Gazebo/RedBright</material>
-  </gazebo>
-  <gazebo reference="RF_link2">
-    <kp>1000000.0</kp>
-    <kd>50.0</kd>
-    <mu1>0.1</mu1>
-    <mu2>0.1</mu2>
-    <maxVel>1.1</maxVel>
-    <minDepth>0.001</minDepth>
-    <fdir1>0 0 0</fdir1>
-    <material>Gazebo/RedBright</material>
-  </gazebo>
-  <gazebo reference="RB_link2">
-    <kp>1000000.0</kp>
-    <kd>50.0</kd>
-    <mu1>0.1</mu1>
-    <mu2>0.1</mu2>
-    <maxVel>1.0</maxVel>
-    <minDepth>0.001</minDepth>
-    <fdir1>0 0 0</fdir1>
-    <material>Gazebo/RedBright</material>
-  </gazebo>
-<!-- Link3 : DarkGrey -->
-  <gazebo reference="LF_link3">
-    <kp>1000000.0</kp>
-    <kd>50.0</kd>
-    <mu1>0.1</mu1>
-    <mu2>0.1</mu2>
-    <maxVel>1.0</maxVel>
-    <minDepth>0.001</minDepth>
-    <fdir1>0 0 0</fdir1>
-    <material>Gazebo/DarkGrey</material>
-  </gazebo>
-  <gazebo reference="LB_link3">
-    <kp>1000000.0</kp>
-    <kd>50.0</kd>
-    <mu1>0.1</mu1>
-    <mu2>0.1</mu2>
-    <maxVel>1.0</maxVel>
-    <minDepth>0.001</minDepth>
-    <fdir1>0 0 0</fdir1>
-    <material>Gazebo/DarkGrey</material>
-  </gazebo>
-  <gazebo reference="RF_link3">
-    <kp>1000000.0</kp>
-    <kd>50.0</kd>
-    <mu1>0.1</mu1>
-    <mu2>0.1</mu2>
-    <maxVel>1.0</maxVel>
-    <minDepth>0.001</minDepth>
-    <fdir1>0 0 0</fdir1>
-    <material>Gazebo/DarkGrey</material>
-  </gazebo>
-  <gazebo reference="RB_link3">
-    <kp>1000000.0</kp>
-    <kd>50.0</kd>
-    <mu1>0.1</mu1>
-    <mu2>0.1</mu2>
-    <maxVel>1.0</maxVel>
-    <minDepth>0.001</minDepth>
-    <fdir1>0 0 0</fdir1>
-    <material>Gazebo/DarkGrey</material>
-  </gazebo>
+  <xacro:macro name="RefLink1" params="ref">
+    <gazebo reference="${ref}">
+      <kp>1000000.0</kp>
+      <kd>50.0</kd>
+      <mu1>0.1</mu1>
+      <mu2>0.1</mu2>
+      <maxVel>1.0</maxVel>
+      <minDepth>0.001</minDepth>
+      <fdir1>0 0 0</fdir1>
+      <material>Gazebo/DarkGrey</material>
+    </gazebo>
+  </xacro:macro>
+  <xacro:macro name="RefLink2" params="ref">
+    <gazebo reference="${ref}">
+      <kp>1000000.0</kp>
+      <kd>50.0</kd>
+      <mu1>0.1</mu1>
+      <mu2>0.1</mu2>
+      <maxVel>1.0</maxVel>
+      <minDepth>0.001</minDepth>
+      <fdir1>0 0 0</fdir1>
+      <material>Gazebo/RedBright</material>
+    </gazebo>
+  </xacro:macro>
+  <xacro:macro name="RefLink3" params="ref">
+    <gazebo reference="${ref}">
+      <kp>1000000.0</kp>
+      <kd>50.0</kd>
+      <mu1>0.1</mu1>
+      <mu2>0.1</mu2>
+      <maxVel>1.0</maxVel>
+      <minDepth>0.001</minDepth>
+      <fdir1>0 0 0</fdir1>
+      <material>Gazebo/DarkGrey</material>
+    </gazebo>
+  </xacro:macro>
   <xacro:macro name="RefJoint" params="ref">
     <gazebo reference="${ref}">
@@ -175,4 +88,16 @@
     </plugin>
   </xacro:macro>
+  <RefLink1 ref="LF_link1"/>
+  <RefLink1 ref="LB_link1"/>
+  <RefLink1 ref="RF_link1"/>
+  <RefLink1 ref="RB_link1"/>
+  <RefLink2 ref="LF_link2"/>
+  <RefLink2 ref="LB_link2"/>
+  <RefLink2 ref="RF_link2"/>
+  <RefLink2 ref="RB_link2"/>
+  <RefLink3 ref="LF_link3"/>
+  <RefLink3 ref="LB_link3"/>
+  <RefLink3 ref="RF_link3"/>
+  <RefLink3 ref="RB_link3"/>
   <RefJoint ref="LF_joint1"/>
   <RefJoint ref="LF_joint2"/>
